File: VGA_SRAM_Shield/VGA_SRAM_Shield.kicad_sch (KiCad schematic)
At the start: 42 parts, among them J1 DIAG, J2 KEYBOARD, J3 DE15_Receptacle_HighDensity, J4 PWR, U1 K6X8008T2B-TF55, U10 74LS161, U11 74LS377, U12 74LS377, U13 74HC245, U14 74HC245, U15 74LS51, U16 74LS08, U2 74HC245, U3 74LS161, U4 74LS161, U5 74LS161, U6 74LS161, U7 74LS161, U8 GAL22V10, U9 GAL22V10, X1 TCXO-14

Commit message: added documentation. gerber of v1.0.0
Parts:
- removed D1: LED_ACTIVITY, symbol Device:LED_Small
- removed J2: KEYBOARD, symbol Connector:Mini-DIN-6
- removed J4: PWR, symbol Connector_Generic:Conn_01x02
- removed R9: R470, symbol Device:R_Small
- removed U11, U12: 74LS377, symbol 74xx:74LS377
- removed U15: 74LS51, symbol 74xx:74LS51
- added C6, C9: C_Small, Capacitor_Tantalum_SMD:CP_EIA-7132-28_AVX-C, symbol Device:C_Small
- added J2: PWR AUX, Connector_PinSocket_2.54mm:PinSocket_2x02_P2.54mm_Vertical, symbol Connector_Generic:Conn_02x02_Counter_Clockwise
- added J5: USB_A, Connector_USB:USB_A_Molex_67643_Horizontal, symbol Connector:USB_A
- added U11, U12, U18, U20: 74HC245, Package_SO:SOP-20_7.5x12.8mm_P1.27mm, symbol 74xx:74HC245
- added U15: 74LS32, Package_SO:SO-14_3.9x8.65mm_P1.27mm, symbol 74xx:74LS32
- added U17: 74HC00, Package_SO:SO-14_3.9x8.65mm_P1.27mm, symbol 74xx:74HC00
- added U19: 74HC14, Package_SO:SO-14_3.9x8.65mm_P1.27mm, symbol 74xx:74HC14
- A1: footprint PCM_arduino-library:Arduino_Due_Shield -> arduino-library:Arduino_Due_Shield
- C1, C2, C3, C4, C5, C7, C8: footprint (none) -> Capacitor_SMD:C_0805_2012Metric
- J1: footprint (none) -> Connector_PinSocket_2.54mm:PinSocket_2x04_P2.54mm_Vertical
- J3: footprint (none) -> Connector_Dsub:DSUB-15-HD_Female_Horizontal_P2.29x1.98mm_EdgePinOffset8.35mm_Housed_MountingHolesOffset10.89mm
- R1, R10, R11, R12, R2, R3, R4, R5, R6, R7, R8: footprint (none) -> Resistor_SMD:R_0805_2012Metric
- U10, U3, U4, U5, U6, U7: footprint (none) -> Package_SO:SO-16_3.9x9.9mm_P1.27mm
- U13, U14, U2: footprint (none) -> Package_SO:SOP-20_7.5x12.8mm_P1.27mm
- U16: footprint (none) -> Package_SO:SO-14_3.9x8.65mm_P1.27mm
- U8, U9: footprint (none) -> Package_DIP:DIP-24_W10.16mm_Socket
Connections:
- net A0: now also U10.14 (Q0), U14.2 (A0); no longer U3.14 (Q0)
- net A1: now also U10.13 (Q1), U14.3 (A1); no longer U3.13 (Q1)
- net A10: now also U13.4 (A2), U5.13 (Q1), U9.2 (I2); no longer U6.14 (Q0), U9.5 (I5)
- net A11: now also U13.5 (A3), U5.12 (Q2), U9.3 (I3); no longer U6.13 (Q1), U9.6 (I6)
- net A12: now also U13.6 (A4), U5.11 (Q3), U9.4 (I4); no longer U6.12 (Q2), U9.7 (I7)
- net A13: now also U13.7 (A5), U6.14 (Q0), U9.5 (I5); no longer U6.11 (Q3), U9.8 (I8)
- net A14: now also U13.8 (A6), U6.13 (Q1), U9.6 (I6); no longer U7.14 (Q0), U9.9 (I9)
- net A15: now also U13.9 (A7), U6.12 (Q2), U9.7 (I7); no longer U7.13 (Q1), U9.10 (I10)
- net A2: now also U10.12 (Q2), U14.4 (A2); no longer U3.12 (Q2)
- net A3: now also U10.11 (Q3), U14.5 (A3); no longer U3.11 (Q3)
- net A4: now also U14.6 (A4), U3.14 (Q0); no longer U4.14 (Q0)
- net A5: now also U14.7 (A5), U3.13 (Q1); no longer U4.13 (Q1)
- net A6: now also U14.8 (A6), U3.12 (Q2); no longer U4.12 (Q2)
- net A7: now also U14.9 (A7), U3.11 (Q3); no longer U4.11 (Q3)
- net A8: now also U13.2 (A0), U4.14 (Q0), U8.9 (I9); no longer U5.12 (Q2), U9.3 (I3)
- net A9: now also U13.3 (A1), U4.13 (Q1), U8.10 (I10); no longer U5.11 (Q3), U9.4 (I4)
- net GND: now also C6.1, C9.1, J2.3 (Pin_3), J2.4 (Pin_4), J5.4 (GND), J5.5 (Shield), U11.10 (GND), U12.10 (GND), U15.7 (GND), U17.7 (GND), U18.10 (GND), U19.7 (GND), U20.10 (GND)
- net H_CLK: now also U10.2 (CP), X1.8 (OUT); no longer U10.14 (Q0)
- net MEMADDR0: now also U11.18 (B0); no longer A1.D22
- net MEMADDR1: now also U11.17 (B1); no longer A1.D23
- net MEMADDR10: now also U12.16 (B2); no longer A1.D32
- net MEMADDR11: now also U12.15 (B3); no longer A1.D33
- net MEMADDR12: now also U12.14 (B4); no longer A1.D34
- net MEMADDR13: now also U12.13 (B5); no longer A1.D35
- net MEMADDR14: now also U12.12 (B6); no longer A1.D36
- net MEMADDR15: now also U12.11 (B7); no longer A1.D37
- net MEMADDR16: now also U18.18 (B0), U20.18 (B0); no longer A1.D38
- net MEMADDR17: now also U18.17 (B1), U20.17 (B1); no longer A1.D39
- net MEMADDR18: now also U18.16 (B2), U20.16 (B2); no longer A1.D40
- net MEMADDR19: now also U18.15 (B3); no longer A1.D41
- net MEMADDR2: now also U11.16 (B2); no longer A1.D24
- net MEMADDR3: now also U11.15 (B3); no longer A1.D25
- net MEMADDR4: now also U11.14 (B4); no longer A1.D26
- net MEMADDR5: now also U11.13 (B5); no longer A1.D27
- net MEMADDR6: now also U11.12 (B6); no longer A1.D28
- net MEMADDR7: now also U11.11 (B7); no longer A1.D29
- net MEMADDR8: now also U12.18 (B0); no longer A1.D30
- net MEMADDR9: now also U12.17 (B1); no longer A1.D31
- net PWR: now also C6.2, C9.2, J2.1 (Pin_1), J2.2 (Pin_2), J5.1 (VBUS), U11.1 (A->B), U11.20 (VCC), U12.1 (A->B), U12.20 (VCC), U15.14 (VCC), U17.14 (VCC), U18.1 (A->B), U18.20 (VCC), U19.14 (VCC), U20.1 (A->B), U20.20 (VCC); no longer U3.10 (CET)
- net ~{SCREEN_VISIBLE}: now also U15.2; no longer U16.5
- net ~{VGA_OUT}: now also U15.3; no longer U13.19 (CE), U14.19 (CE), U16.6
- net at A1.D11: no longer U16.1
- net at U1.17 (~{WE}): now also U16.10, U19.6; no longer A1.D12
- net at U16.4: no longer U16.2
- net at R4.1: now also U2.13 (B5); no longer U2.15 (B3)
- net at A1.D18 (D18/TX1): now also J5.2 (D-)
- net at A1.D19 (D19/RX1): now also J5.3 (D+)
- net at U10.15 (TC): now also U3.10 (CET)
- net at U2.11 (B7): now also R7.1; no longer R8.1
- net at U2.12 (B6): now also R8.1; no longer R7.1
- net at R6.1: now also U2.15 (B3); no longer U2.13 (B5)
- net at U2.16 (B2): now also R1.1; no longer R3.1
- net at U2.18 (B0): now also R3.1; no longer R1.1
- net DATA7: now reaches U1.9 (I/O1), U2.2 (A0)
- net DATA7: now also A1.D40; no longer A1.D49
- net DATA6: now reaches U1.10 (I/O2), U2.3 (A1)
- net DATA6: now also A1.D39; no longer A1.D48
- net DATA5: now reaches U1.13 (I/O3), U2.4 (A2)
- net DATA5: now also A1.D38; no longer A1.D47
- net DATA4: now reaches U1.14 (I/O4), U2.5 (A3)
- net DATA4: now also A1.D37; no longer A1.D46
- net DATA3: now reaches U1.31 (I/O5), U2.6 (A4)
- net DATA3: now also A1.D36; no longer A1.D45
- net DATA2: now reaches U1.32 (I/O6), U2.7 (A5)
- net DATA2: now also A1.D35; no longer A1.D44
- net DATA1: now reaches U1.35 (I/O7), U2.8 (A6)
- net DATA1: now also A1.D34; no longer A1.D43
- net DATA0: now reaches U1.36 (I/O8), U2.9 (A7)
- net DATA0: now also A1.D33; no longer A1.D42
- net at U16.8: now also U17.5
- net at U16.9: now also U11.19 (CE), U12.19 (CE), U18.19 (CE), U19.4
- net MCUMEMADDR14: now reaches A1.A10
- net MCUMEMADDR14: now also U12.8 (A6)
- net MCUMEMADDR15: now reaches A1.A11
- net MCUMEMADDR15: now also U12.9 (A7)
- net MCUMEMADDR12: now reaches A1.A8
- net MCUMEMADDR12: now also U12.6 (A4)
- net MCUMEMADDR13: now reaches A1.A9
- net MCUMEMADDR13: now also U12.7 (A5)
- net MCU OE: now reaches A1.D2
- net MCU OE: now also U19.1
- net MCU CE: now reaches A1.D3
- net MCU CE: now also U19.3
- net MCU WE: now reaches A1.D4 (D4_CS1)
- net MCU WE: now also U19.5
- net MCUMEMADDR1: now reaches A1.D50
- net MCUMEMADDR1: now also U11.3 (A1)
- net MCUMEMADDR0: now reaches A1.D51
- net MCUMEMADDR0: now also U11.2 (A0)
- net MCUMEMADDR19: now reaches A1.D6
- net MCUMEMADDR19: now also U18.5 (A3)
- net MCUMEMADDR18: now reaches A1.D7
- net MCUMEMADDR18: now also U18.4 (A2)
- net MCUMEMADDR17: now reaches A1.D8
- net MCUMEMADDR17: now also U18.3 (A1)
- net MCUMEMADDR16: now reaches A1.D9
- net MCUMEMADDR16: now also U18.2 (A0)
- new net A16: U20.2 (A0), U6.11 (Q3), U9.8 (I8)
- new net A17: U20.3 (A1), U7.14 (Q0), U9.9 (I9)
- new net A18: U20.4 (A2), U7.13 (Q1), U9.10 (I10)
- new net MCUMEMADDR10: A1.D27, U12.4 (A2)
- new net MCUMEMADDR11: A1.D28, U12.5 (A3)
- new net MCUMEMADDR2: A1.D49, U11.4 (A2)
- new net MCUMEMADDR3: A1.D48, U11.5 (A3)
- new net MCUMEMADDR4: A1.D47, U11.6 (A4)
- new net MCUMEMADDR5: A1.D46, U11.7 (A5)
- new net MCUMEMADDR6: A1.D45, U11.8 (A6)
- new net MCUMEMADDR7: A1.D44, U11.9 (A7)
- new net MCUMEMADDR8: A1.D25, U12.2 (A0)
- new net MCUMEMADDR9: A1.D26, U12.3 (A1)
- new net ~{MCU OE}: U16.1, U17.4, U19.2
- new net ~{TIMING ADDR}: U13.19 (CE), U14.19 (CE), U15.1, U16.2, U17.6, U20.19 (CE)
- no-connect marks 118 -> 150
Other:
- moved on the sheet: A1, C1, C2, C3, C4, C5, C7, C8, J1, J3, R1, R10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

Commit message: v1.12
Parts:
- R2: value R900 -> R800
- R3: value R1.5K -> R1.8K
- R4: value R470 -> R2.2K
- R5: value R900 -> R470
- R6: value R1.5K -> R1.2K
- R8: value R900 -> R1.8K
- U8, U9: footprint Package_DIP:DIP-24_W10.16mm_Socket -> Package_DIP:DIP-24_W7.62mm_Socket
Connections:
- net PWR: now also U5.10 (CET)
- net at J3.2, R5.2, R6.2: now also R3.2; no longer R4.2
- net at U4.15 (TC): no longer U5.10 (CET)
- net at U2.16 (B2): now also R3.1; no longer R1.1
- net at U2.17 (B1): now also R1.1; no longer R2.1
- net at U2.18 (B0): now also R2.1; no longer R3.1
- net at R1.2, R2.2: now also J3.3; no longer J3.1, R3.2
- net at R7.2, R8.2: now also J3.1, R4.2; no longer J3.3
Other:
- moved on the sheet: R1, R2, R3

Commit message: new shield v1.1
Parts:
- removed C1, C4: 560pf, Capacitor_SMD:C_0805_2012Metric, symbol Device:C_Small
- removed C6: C_Small, Capacitor_Tantalum_SMD:CP_EIA-7132-28_AVX-C, symbol Device:C_Small
- removed J1: DIAG, Connector_PinSocket_2.54mm:PinSocket_2x04_P2.54mm_Vertical, symbol Connector_Generic:Conn_02x04_Counter_Clockwise
- removed R10: R10K, Resistor_SMD:R_0805_2012Metric, symbol Device:R_Small
- C9: footprint Capacitor_Tantalum_SMD:CP_EIA-7132-28_AVX-C -> Capacitor_SMD:CP_Elec_4x4.5
Connections:
- net GND: now also C9.2, U1.6 (~{CS1}); no longer C9.1
- net H_VISIBLE: now also A1.D14 (D14/TX3)
- net PWR: now also C9.1; no longer C9.2
- net ~{SCREEN_VISIBLE}: now also A1.D10 (D10_CS0)
- net ~{V_VISIBLE}: now also A1.D15 (D15/RX3)
- no-connect marks 150 -> 145
Other:
- moved on the sheet: C7, C9, J5
