File: VGA_SRAM_Shield/VGA_SRAM_Shield.kicad_sch (KiCad schematic)
At the start: 42 parts, among them J1 CONN_ADDR_MEM, J2 PWR AUX, J3 DE15_Receptacle_HighDensity, J5 USB_A, U1 K6X8008T2B-TF55, U10 74LS161, U11 74HC245, U12 74HC245, U13 74HC245, U14 74HC245, U15 74LS32, U16 74LS08, U17 74HC00, U18 74HC245, U19 74HC14, U2 74HC245, U20 74HC245, U3 74LS161, U4 74LS161, U5 74LS161, U6 74LS161, U7 74LS161, U8 GAL22V10, U9 GAL22V10, X1 TCXO-14

Commit message: wip
Parts:
- removed J1: CONN_ADDR_MEM, Connector_PinHeader_1.27mm:PinHeader_2x10_P1.27mm_Vertical, symbol Connector_Generic:Conn_02x10_Counter_Clockwise
- removed J5: USB_A, Connector_USB:USB_A_Molex_67643_Horizontal, symbol Connector:USB_A
- added C1: 4.7nF, Capacitor_SMD:C_0805_2012Metric, symbol Device:C_Small
- added J1: ANALOG, Connector_PinSocket_2.54mm:PinSocket_2x05_P2.54mm_Vertical, symbol Connector_Generic:Conn_02x05_Counter_Clockwise
- added J4: Micro_SD_Card, SDCard:J_SD_Card-micro_socket_A, symbol Connector:Micro_SD_Card
- added J5: USB_A_Stacked, Connector_USB:USB_A_CUI_UJ2-ADH-TH_Horizontal_Stacked, symbol Connector:USB_A_Stacked
- added J6: AUDIO, Connector_PinSocket_2.54mm:PinSocket_1x03_P2.54mm_Vertical, symbol Connector:Conn_01x03_Pin
- added J7: DIGITAL, Connector_PinSocket_2.54mm:PinSocket_2x05_P2.54mm_Vertical, symbol Connector_Generic:Conn_02x05_Counter_Clockwise
- added J8: Mini-DIN-6, Libraries:mini-DIN 6, symbol Connector:Mini-DIN-6
- added JP1: JP_RESOLUTION, Connector_PinHeader_2.54mm:PinHeader_1x02_P2.54mm_Vertical, symbol Jumper:Jumper_2_Open
- added R10: R200, Resistor_SMD:R_0805_2012Metric, symbol Device:R_Small
- added R13: R490K, Resistor_SMD:R_0805_2012Metric, symbol Device:R_Small
- added R14: R3.9K, Resistor_SMD:R_0805_2012Metric, symbol Device:R_Small
- added R9: 10K, Resistor_SMD:R_0805_2012Metric, symbol Device:R_Small
Connections:
- net GND: now also A1.GND4 (SPI_GND), C1.2, J1.10 (Pin_10), J4.6 (VSS), J4.9 (SHIELD), J5.4 (GND1), J5.8 (GND2), J5.9 (Shield), J6.1 (Pin_1), J7.10 (Pin_10), J7.9 (Pin_9), J8.3, R9.1
- net H_VISIBLE: now also A1.D24; no longer A1.D9
- net PWR: now also A1.5V2 (SPI_5V), J1.1 (Pin_1), J4.4 (VDD), J5.1 (VBUS1), J5.5 (VBUS2), J8.4, JP1.2 (B)
- net RESOLUTION: now also A1.D5, JP1.1 (A), R10.1, R9.2; no longer A1.D17 (D17/RX2), U8.23 (IO23), U9.23 (IO23)
- net ~{SCREEN_VISIBLE}: now also A1.D22; no longer A1.D16 (D16/TX2)
- net ~{V_VISIBLE}: now also A1.D23; no longer A1.D8
- net at A1.D18 (D18/TX1): now also J5.2 (D1-)
- net at A1.D19 (D19/RX1): now also J5.3 (D1+)
- net 3.3V: now reaches A1.3V3 (3.3V)
- net 3.3V: now also J7.2 (Pin_2)
- net 5V: now reaches A1.5V1 (5V)
- net 5V: now also A1.5V3 (5V), A1.5V4 (5V), J7.1 (Pin_1)
- net at A1.A0: now also J1.2 (Pin_2)
- net at A1.A1: now also J1.3 (Pin_3)
- net DATA13: now reaches A1.A10
- net DATA14: now reaches A1.A11
- net at A1.A2: now also J1.4 (Pin_4)
- net at A1.A3: now also J1.5 (Pin_5)
- net at A1.A4: now also J1.9 (Pin_9)
- net at A1.A5: now also J1.8 (Pin_8)
- net at A1.A6: now also J1.7 (Pin_7)
- net at A1.A7: now also J1.6 (Pin_6)
- net DATA11: now reaches A1.A8
- net DATA12: now reaches A1.A9
- net SD_CS: now reaches A1.D10 (D10_CS0)
- net SD_CS: now also J4.2 (DAT3/CD)
- net D13: now reaches A1.D13
- net D13: now also J7.5 (Pin_5)
- net D31: now reaches A1.D31
- net D31: now also J7.6 (Pin_6)
- net D42: now reaches A1.D42
- net D42: now also J7.7 (Pin_7)
- net D43: now reaches A1.D43
- net D43: now also J7.8 (Pin_8)
- net DATA15: now reaches A1.D52 (D52_CS2)
- net DATA8: now reaches A1.D53
- net at A1.D6: now also R13.1
- net at A1.D7: now also R14.1
- net DATA9: now reaches A1.DAC0
- net DATA10: now reaches A1.DAC1
- net at A1.MISO (SPI_MISO): now also J4.7 (DAT0)
- net at A1.MOSI (SPI_MOSI): now also J4.3 (CMD)
- net at A1.SCK (SPI_SCK): now also J4.5 (CLK)
- new net: R10.2, U8.23 (IO23), U9.23 (IO23)
- new net: C1.1, J6.2 (Pin_2), J6.3 (Pin_3), R13.2, R14.2
- new net: A1.D16 (D16/TX2), J5.6 (D2-), J8.5
- new net: A1.D17 (D17/RX2), J5.7 (D2+), J8.1
- new net D8: A1.D8, J7.3 (Pin_3)
- new net D9: A1.D9, J7.4 (Pin_4)
- no-connect marks 141 -> 109
Other:
- moved on the sheet: A1, C2, C3, C5, C7, C8, C9, J2, J3, R1, R11, R12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
