File: VGA_SRAM_Shield/VGA_SRAM_Shield-backups/VGA_SRAM_Shield-2024-12-04_012755/VGA_SRAM_Shield.kicad_sch (KiCad schematic)
At the start: 42 parts, among them J1 CONN_ADDR_MEM, J2 PWR AUX, J3 DE15_Receptacle_HighDensity, J5 USB_A, U1 K6X8008T2B-TF55, U10 74LS161, U11 74HC245, U12 74HC245, U13 74HC245, U14 74HC245, U15 74LS32, U16 74LS08, U17 74HC00, U18 74HC245, U19 74HC14, U2 74HC245, U20 74HC245, U3 74LS161, U4 74LS161, U5 74LS161, U6 74LS161, U7 74LS161, U8 GAL22V10, U9 GAL22V10, X1 TCXO-14

Commit message: kicad design changes
Parts:
- removed J1: CONN_ADDR_MEM, Connector_PinHeader_1.27mm:PinHeader_2x10_P1.27mm_Vertical, symbol Connector_Generic:Conn_02x10_Counter_Clockwise
- added C1, C4: 560pf, Capacitor_SMD:C_0805_2012Metric, symbol Device:C_Small
- added C6: C_Small, Capacitor_Tantalum_SMD:CP_EIA-7132-28_AVX-C, symbol Device:C_Small
- added J1: DIAG, Connector_PinSocket_2.54mm:PinSocket_2x04_P2.54mm_Vertical, symbol Connector_Generic:Conn_02x04_Counter_Clockwise
- added R10: R10K, Resistor_SMD:R_0805_2012Metric, symbol Device:R_Small
- C9: footprint Capacitor_SMD:CP_Elec_4x4.5 -> Capacitor_Tantalum_SMD:CP_EIA-7132-28_AVX-C
- R2: value R800 -> R900
- R3: value R1.8K -> R1.5K
- R4: value R2.2K -> R470
- R5: value R470 -> R900
- R6: value R1.2K -> R1.5K
- R8: value R1.8K -> R900
- U8, U9: footprint Package_DIP:DIP-24_W7.62mm_Socket -> Package_DIP:DIP-24_W10.16mm_Socket
Connections:
- net DATA0: now also A1.D33; no longer A1.D51
- net DATA1: now also A1.D34; no longer A1.D50
- net DATA2: now also A1.D35; no longer A1.D49
- net DATA3: now also A1.D36; no longer A1.D48
- net DATA4: now also A1.D37; no longer A1.D47
- net DATA5: now also A1.D38; no longer A1.D46
- net DATA6: now also A1.D39; no longer A1.D45
- net DATA7: now also A1.D40; no longer A1.D44
- net GND: now also C9.1, C6.1, J1.5 (Pin_5), R10.1; no longer C9.2, U1.6 (~{CS1})
- net H_VISIBLE: now also J1.2 (Pin_2); no longer A1.D9
- net MCUMEMADDR0: now also A1.D51; no longer A1.D25
- net MCUMEMADDR1: now also A1.D50; no longer A1.D26
- net MCUMEMADDR10: now also A1.D27; no longer A1.D32
- net MCUMEMADDR11: now also A1.D28; no longer A1.D33
- net MCUMEMADDR12: now also A1.A8; no longer A1.D34
- net MCUMEMADDR13: now also A1.A9; no longer A1.D35
- net MCUMEMADDR14: now also A1.A10; no longer A1.D36
- net MCUMEMADDR15: now also A1.A11; no longer A1.D37
- net MCUMEMADDR16: now also A1.D9; no longer A1.D38
- net MCUMEMADDR17: now also A1.D8; no longer A1.D39
- net MCUMEMADDR18: now also A1.D7; no longer A1.D40
- net MCUMEMADDR19: now also A1.D6; no longer A1.D41
- net MCUMEMADDR2: now also A1.D49; no longer A1.D27
- net MCUMEMADDR3: now also A1.D48; no longer A1.D28
- net MCUMEMADDR4: now also A1.D47; no longer A1.D14 (D14/TX3)
- net MCUMEMADDR5: now also A1.D46; no longer A1.D15 (D15/RX3)
- net MCUMEMADDR6: now also A1.D45; no longer A1.D29
- net MCUMEMADDR7: now also A1.D44; no longer A1.D11
- net MCUMEMADDR8: now also A1.D25; no longer A1.D12
- net MCUMEMADDR9: now also A1.D26; no longer A1.D30
- net MEMADDR19: no longer U20.15 (B3)
- net PWR: now also C9.2, C1.1, C4.1, C6.2; no longer C9.1
- net V_FRONT_PORCH: now also C4.2, J1.7 (Pin_7)
- net ~{H_SYNC}: now also J1.1 (Pin_1)
- net ~{SCREEN_VISIBLE}: now also J1.3 (Pin_3); no longer A1.D16 (D16/TX2)
- net ~{V_RESET}: now also J1.4 (Pin_4)
- net ~{V_SYNC}: now also J1.6 (Pin_6)
- net ~{V_VISIBLE}: now also J1.8 (Pin_8); no longer A1.D8
- net at U3.1 (~{MR}), U4.1 (~{MR}), U5.2 (CP)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: now also C1.2
- net at R7.2, R8.2: now also J3.3; no longer J3.1, R4.2
- net at U2.16 (B2): now also R1.1; no longer R3.1
- net at U2.17 (B1): now also R2.1; no longer R1.1
- net at U2.18 (B0): now also R3.1; no longer R2.1
- net at R1.2, R2.2: now also J3.1, R3.2; no longer J3.3
- net at J3.2, R5.2, R6.2: now also R4.2; no longer R3.2
- net A19: no longer names the net of U20.5 (A3)
- net A19: no longer U7.12 (Q2)
- removed net RESOLUTION: A1.D17 (D17/RX2), U8.23 (IO23), U9.23 (IO23)
- new net: R10.2, U1.6 (~{CS1})
- no-connect marks 141 -> 151
Other:
- moved on the sheet: C7, C9, J5, R1, R2, R3, U11, U12, U18
