File: VGA_SRAM_SHIELD_DOUBLE_BUFFER/VGA_SRAM_SHUIELD_DOUBLE_BUFFER.kicad_sch (KiCad schematic)
At the start: 45 parts, among them J1 USB_A_Stacked, J2 ANALOG, J3 Mini-DIN-6, J4 PWR AUX, J5 ISP, J6 Micro_SD_Card, J7 VGA D-SUB15, J8 AUDIO, U1 74HC245, U10 74HC245, U11 74HC245, U12 74LS08, U13 74LS32, U14 DATA_BANK1, U15 DATA_BANK2, U16 74HC245, U17 74HC245, U18 74HC245, U19 K6X8008T2B-TF55, U2 74HC245, U20 K6X8008T2B-TF55, U21 74HC245, U22 74HC245, U3 74HC245, U4 ATF1504AS, U5 74HC245, U6 74HC245, U7 74HC245, U8 74HC14, U9 74HC245, X1 TCXO-14

Commit message: updates to double buffer and multiplexed, 2xatf1508 concept
Connections:
- net BANK_SELECT: now also A1.D5
- net DATA_BANK10: now also U19.9 (I/O1), U21.2 (A0); no longer U19.36 (I/O8), U21.9 (A7)
- net DATA_BANK11: now also U19.10 (I/O2), U21.3 (A1); no longer U19.35 (I/O7), U21.8 (A6)
- net DATA_BANK12: now also U19.13 (I/O3), U21.4 (A2); no longer U19.32 (I/O6), U21.7 (A5)
- net DATA_BANK13: now also U19.14 (I/O4), U21.5 (A3); no longer U19.31 (I/O5), U21.6 (A4)
- net DATA_BANK14: now also U19.31 (I/O5), U21.6 (A4); no longer U19.14 (I/O4), U21.5 (A3)
- net DATA_BANK15: now also U19.32 (I/O6), U21.7 (A5); no longer U19.13 (I/O3), U21.4 (A2)
- net DATA_BANK16: now also U19.35 (I/O7), U21.8 (A6); no longer U19.10 (I/O2), U21.3 (A1)
- net DATA_BANK17: now also U19.36 (I/O8), U21.9 (A7); no longer U19.9 (I/O1), U21.2 (A0)
- net DATA_BANK20: now also U20.9 (I/O1), U22.2 (A0); no longer U20.36 (I/O8), U22.9 (A7)
- net DATA_BANK21: now also U20.10 (I/O2), U22.3 (A1); no longer U20.35 (I/O7), U22.8 (A6)
- net DATA_BANK22: now also U20.13 (I/O3), U22.4 (A2); no longer U20.32 (I/O6), U22.7 (A5)
- net DATA_BANK23: now also U20.14 (I/O4), U22.5 (A3); no longer U20.31 (I/O5), U22.6 (A4)
- net DATA_BANK24: now also U20.31 (I/O5), U22.6 (A4); no longer U20.14 (I/O4), U22.5 (A3)
- net DATA_BANK25: now also U20.32 (I/O6), U22.7 (A5); no longer U20.13 (I/O3), U22.4 (A2)
- net DATA_BANK26: now also U20.35 (I/O7), U22.8 (A6); no longer U20.10 (I/O2), U22.3 (A1)
- net DATA_BANK27: now also U20.36 (I/O8), U22.9 (A7); no longer U20.9 (I/O1), U22.2 (A0)
- no-connect marks 69 -> 68
Other:
- note added: "Memory and color output"
